Commit message: Added moveit configuration for arm with separator

File: schunk_lwa4p_description/urdf/lwa4p/lwa4p_arm.xacro (robot description, xacro)
@@ -2,10 +2,10 @@
 <robot xmlns:xacro="http://www.ros.org/wiki/xacro" name="lwa4p">
   <xacro:macro name="lwa4p_arm" params="parent arm_id *origin has_podest">
-    <xacro:include filename="$(find schunk_lwa4p_moveit)/urdf/common.xacro"/>
+    <xacro:include filename="$(find schunk_lwa4p_description)/urdf/common.xacro"/>
     <xacro:property name="safety_offset" value="0.02"/>
     <xacro:arg name="gazebo" default="true"/>
     <xacro:if value="$(arg gazebo)">
       <!-- Gazebo Tags -->
-      <xacro:include filename="$(find schunk_lwa4p_moveit)/urdf/lwa4p/lwa4p_arm.gazebo.xacro"/>
+      <xacro:include filename="$(find schunk_lwa4p_description)/urdf/lwa4p/lwa4p_arm.gazebo.xacro"/>
     </xacro:if>
      <xacro:if value="${has_podest}">
@@ -21,5 +21,5 @@
           <origin xyz="0 0 0" rpy="0 ${M_PI} 0" />
           <geometry>
-            <mesh filename="package://schunk_lwa4p_moveit/meshes/lwa4p/stl/arm_base_link.stl" />
+            <mesh filename="package://schunk_lwa4p_description/meshes/lwa4p/stl/arm_base_link.stl" />
           </geometry>
            <material name="Schunk/DarkGrey" />
@@ -28,5 +28,5 @@
           <origin xyz="0 0 0" rpy="0 ${M_PI} 0" />
           <geometry>
-          <mesh filename="package://schunk_lwa4p_moveit/meshes/lwa4p/stl/arm_base_link.stl" />
+          <mesh filename="package://schunk_lwa4p_description/meshes/lwa4p/stl/arm_base_link.stl" />
           </geometry>
         </collision>
@@ -60,5 +60,5 @@
         <origin xyz="0 0 0" rpy="0 0 0" />
         <geometry>
-          <mesh filename="package://schunk_lwa4p_moveit/meshes/lwa4p/stl/arm_1_link.stl" />
+          <mesh filename="package://schunk_lwa4p_description/meshes/lwa4p/stl/arm_1_link.stl" />
         </geometry>
         <material name="Schunk/Blue" />
@@ -67,5 +67,5 @@
         <origin xyz="0 0 0" rpy="0 0 0" />
         <geometry>
-          <mesh filename="package://schunk_lwa4p_moveit/meshes/lwa4p/stl/arm_1_link.stl" />
+          <mesh filename="package://schunk_lwa4p_description/meshes/lwa4p/stl/arm_1_link.stl" />
         </geometry>
       </collision>
@@ -91,12 +91,12 @@
         <origin xyz="0 0 0" rpy="0 0 0" />
         <geometry>
-          <mesh filename="package://schunk_lwa4p_moveit/meshes/lwa4p/stl/arm_2_link.stl" />
-        </geometry>
-        <material name="Schunk/LightGrey" />
-      </visual>
-      <collision>
-        <origin xyz="0 0 0" rpy="0 0 0" />
-        <geometry>
-          <mesh filename="package://schunk_lwa4p_moveit/meshes/lwa4p/stl/arm_2_link.stl" />
+          <mesh filename="package://schunk_lwa4p_description/meshes/lwa4p/stl/arm_2_link.stl" />
+        </geometry>
+        <material name="Schunk/LightGrey" />
+      </visual>
+      <collision>
+        <origin xyz="0 0 0" rpy="0 0 0" />
+        <geometry>
+          <mesh filename="package://schunk_lwa4p_description/meshes/lwa4p/stl/arm_2_link.stl" />
         </geometry>
       </collision>
@@ -123,12 +123,12 @@
         <origin xyz="0 0 0" rpy="0 0 0" />
         <geometry>
-          <mesh filename="package://schunk_lwa4p_moveit/meshes/lwa4p/stl/arm_3_link.stl" />
-        </geometry>
-        <material name="Schunk/LightGrey" />
-      </visual>
-      <collision>
-        <origin xyz="0 0 0" rpy="0 0 0" />
-        <geometry>
-          <mesh filename="package://schunk_lwa4p_moveit/meshes/lwa4p/stl/arm_3_link.stl" />
+          <mesh filename="package://schunk_lwa4p_description/meshes/lwa4p/stl/arm_3_link.stl" />
+        </geometry>
+        <material name="Schunk/LightGrey" />
+      </visual>
+      <collision>
+        <origin xyz="0 0 0" rpy="0 0 0" />
+        <geometry>
+          <mesh filename="package://schunk_lwa4p_description/meshes/lwa4p/stl/arm_3_link.stl" />
         </geometry>
       </collision>
@@ -155,12 +155,12 @@
         <origin xyz="0 0 0" rpy="0 0 0" />
         <geometry>
-          <mesh filename="package://schunk_lwa4p_moveit/meshes/lwa4p/stl/arm_4_link.stl" />
-        </geometry>
-        <material name="Schunk/LightGrey" />
-      </visual>
-      <collision>
-        <origin xyz="0 0 0" rpy="0 0 0" />
-        <geometry>
-          <mesh filename="package://schunk_lwa4p_moveit/meshes/lwa4p/stl/arm_4_link.stl" />
+          <mesh filename="package://schunk_lwa4p_description/meshes/lwa4p/stl/arm_4_link.stl" />
+        </geometry>
+        <material name="Schunk/LightGrey" />
+      </visual>
+      <collision>
+        <origin xyz="0 0 0" rpy="0 0 0" />
+        <geometry>
+          <mesh filename="package://schunk_lwa4p_description/meshes/lwa4p/stl/arm_4_link.stl" />
         </geometry>
       </collision>
@@ -187,5 +187,5 @@
         <origin xyz="0 0 0" rpy="0 0 0" />
         <geometry>
-          <mesh filename="package://schunk_lwa4p_moveit/meshes/lwa4p/stl/arm_5_link.stl" />
+          <mesh filename="package://schunk_lwa4p_description/meshes/lwa4p/stl/arm_5_link.stl" />
         </geometry>
         <material name="Schunk/Blue" />
@@ -194,5 +194,5 @@
         <origin xyz="0 0 0" rpy="0 0 0" />
         <geometry>
-          <mesh filename="package://schunk_lwa4p_moveit/meshes/lwa4p/stl/arm_5_link.stl" />
+          <mesh filename="package://schunk_lwa4p_description/meshes/lwa4p/stl/arm_5_link.stl" />
         </geometry>
       </collision>
@@ -219,12 +219,12 @@
         <origin xyz="0 0 0" rpy="0 0 0" />
         <geometry>
-          <mesh filename="package://schunk_lwa4p_moveit/meshes/lwa4p/stl/arm_6_link.stl" />
-        </geometry>
-        <material name="Schunk/LightGrey" />
-      </visual>
-      <collision>
-        <origin xyz="0 0 0" rpy="0 0 0" />
-        <geometry>
-          <mesh filename="package://schunk_lwa4p_moveit/meshes/lwa4p/stl/arm_6_link.stl" />
+          <mesh filename="package://schunk_lwa4p_description/meshes/lwa4p/stl/arm_6_link.stl" />
+        </geometry>
+        <material name="Schunk/LightGrey" />
+      </visual>
+      <collision>
+        <origin xyz="0 0 0" rpy="0 0 0" />
+        <geometry>
+          <mesh filename="package://schunk_lwa4p_description/meshes/lwa4p/stl/arm_6_link.stl" />
         </geometry>
       </collision>

File: schunk_lwa4p_description/urdf/lwa4p/lwa4p_arm_separator.urdf.xacro (robot description, xacro)
@@ -6,5 +6,7 @@
   	<xacro:arg name="gazebo" value="${gazebo}"/>
   </xacro:include>
-  <xacro:include filename="$(find schunk_lwa4p_description)/urdf/tools/separator.xacro"/>
+  <xacro:include filename="$(find schunk_lwa4p_description)/urdf/tools/separator.xacro" >
+	<xacro:arg name="gazebo" value="${gazebo}"/>
+  </xacro:include>
 	<link name="world">
 	</link>

File: schunk_lwa4p_description/urdf/tools/separator.xacro (robot description, xacro)
@@ -27,5 +27,5 @@
             <inertial>
                 <origin rpy="0 0 0" xyz="0 0 0"/>
-                <mass value="10" />
+                <mass value="2.5" />
                 <inertia ixx="1" ixy="0.0" ixz="0.0" iyy="1" iyz="0.0" izz="1"/>
             </inertial>

Commit message: Added dynamics damping and friction, added joint remapping, removed link colors

File: schunk_lwa4p_description/urdf/lwa4p/lwa4p_arm.xacro (robot description, xacro)
@@ -4,4 +4,6 @@
     <xacro:include filename="$(find schunk_lwa4p_description)/urdf/common.xacro"/>
     <xacro:property name="safety_offset" value="0.02"/>
+    <xacro:property name="dynamics_damping" value="0.5"/>
+    <xacro:property name="dynamics_friction" value="0.5"/>
     <xacro:arg name="gazebo" default="true"/>
     <xacro:if value="$(arg gazebo)">
@@ -62,5 +64,5 @@
           <mesh filename="package://schunk_lwa4p_description/meshes/lwa4p/stl/arm_1_link.stl" />
         </geometry>
-        <material name="Schunk/Blue" />
+        <!--material name="Schunk/Blue" /-->
       </visual>
       <collision>
@@ -77,4 +79,5 @@
       <child link="${arm_id}_link1"/>
       <axis xyz="0 0 1"/>
+      <dynamics damping="${dynamics_damping}" friction="${dynamics_friction}"/>
       <limit effort="370" velocity="1.26" lower="${-2.967 + safety_offset}" upper="${2.967 - safety_offset}"/>
       <safety_controller k_position="20" k_velocity="50" soft_lower_limit="${-6.28 + 0.01}" soft_upper_limit="${6.28 - 0.01}"/>
@@ -93,5 +96,5 @@
           <mesh filename="package://schunk_lwa4p_description/meshes/lwa4p/stl/arm_2_link.stl" />
         </geometry>
-        <material name="Schunk/LightGrey" />
+        <!--material name="Schunk/LightGrey" /-->
       </visual>
       <collision>
@@ -106,7 +109,8 @@
     <joint name="${arm_id}_joint2" type="revolute">
       <origin xyz="0 0 0" rpy="1.5708 0 0"/>
->      <parent link="${arm_id}_link1"/>
+      <parent link="${arm_id}_link1"/>
       <child link="${arm_id}_link2"/>
       <axis xyz="0 0 1"/>
+      <dynamics damping="${dynamics_damping}" friction="${dynamics_friction}"/>
       <limit effort="370" velocity="1.26" lower="${-2.967 + safety_offset}" upper="${2.967 - safety_offset}"/>
       <safety_controller k_position="20" k_velocity="50" soft_lower_limit="${-2.09 + 0.01}" soft_upper_limit="${2.09 - 0.01}" />
@@ -125,5 +129,5 @@
           <mesh filename="package://schunk_lwa4p_description/meshes/lwa4p/stl/arm_3_link.stl" />
         </geometry>
-        <material name="Schunk/LightGrey" />
+        <!--material name="Schunk/LightGrey" /-->
       </visual>
       <collision>
@@ -141,4 +145,5 @@
       <child link="${arm_id}_link3"/>
       <axis xyz="0 0 1"/>
+      <dynamics damping="${dynamics_damping}" friction="${dynamics_friction}"/>
       <limit effort="176" velocity="1.26" lower="${-2.714 + safety_offset}" upper="${2.714 - safety_offset}"/>
       <safety_controller k_position="20" k_velocity="25" soft_lower_limit="${-6.28 + 0.01}" soft_upper_limit="${6.28 - 0.01}" />
@@ -157,5 +162,5 @@
           <mesh filename="package://schunk_lwa4p_description/meshes/lwa4p/stl/arm_4_link.stl" />
         </geometry>
-        <material name="Schunk/LightGrey" />
+        <!--material name="Schunk/LightGrey" /-->
       </visual>
       <collision>
@@ -173,4 +178,5 @@
       <child link="${arm_id}_link4"/>
       <axis xyz="0 0 1" />
+      <dynamics damping="${dynamics_damping}" friction="${dynamics_friction}"/>
       <limit effort="176" velocity="1.26" lower="${-2.967 + safety_offset}" upper="${2.967 - safety_offset}"/>
       <safety_controller k_position="20" k_velocity="25" soft_lower_limit="${-2.09 + 0.01}" soft_upper_limit="${2.09 - 0.01}" />
@@ -189,5 +195,5 @@
           <mesh filename="package://schunk_lwa4p_description/meshes/lwa4p/stl/arm_5_link.stl" />
         </geometry>
-        <material name="Schunk/Blue" />
+        <!--material name="Schunk/Blue" /-->
       </visual>
       <collision>
@@ -205,4 +211,5 @@
       <child link="${arm_id}_link5"/>
       <axis xyz="0 0 1" />
+      <dynamics damping="${dynamics_damping}" friction="${dynamics_friction}"/>
       <limit effort="41.6" velocity="1.26" lower="${-2.967 + safety_offset}" upper="${2.967 - safety_offset}" />
       <safety_controller k_position="20" k_velocity="25" soft_lower_limit="${-6.28 + 0.01}" soft_upper_limit="${6.28 - 0.01}" />
@@ -221,5 +228,5 @@
           <mesh filename="package://schunk_lwa4p_description/meshes/lwa4p/stl/arm_6_link.stl" />
         </geometry>
-        <material name="Schunk/LightGrey" />
+        <!--material name="Schunk/LightGrey" /-->
       </visual>
       <collision>
@@ -237,4 +244,5 @@
       <child link="${arm_id}_link6"/>
       <axis xyz="0 0 1" />
+      <dynamics damping="${dynamics_damping}" friction="${dynamics_friction}"/>
       <limit effort="20.1" velocity="1.26" lower="${-2.967 + safety_offset}" upper="${2.967 - safety_offset}" />
       <safety_controller k_position="20" k_velocity="25" soft_lower_limit="${-2.09 + 0.01}" soft_upper_limit="${2.09 - 0.01}" />

File: schunk_lwa4p_description/urdf/lwa4p/lwa4p_arm_separator.gazebo.xacro (robot description, xacro)
@@ -11,20 +11,20 @@
     <gravity>true</gravity>
       <self_collide>false</self_collide>
-      <material value="Gazebo/LightGrey" />
+      <!--material value="Gazebo/LightGrey" /-->
   </gazebo>
   <gazebo reference="${arm_id}_link2">
     <gravity>true</gravity>
     <self_collide>false</self_collide>
-    <material value="Gazebo/Blue" />
+    <!--material value="Gazebo/Blue" /-->
   </gazebo>
   <gazebo reference="${arm_id}_link3">
     <gravity>true</gravity>
     <self_collide>false</self_collide>
-    <material value="Gazebo/LightGrey" />
+    <!--material value="Gazebo/LightGrey" /-->
   </gazebo>
   <gazebo reference="${arm_id}_link4">
     <gravity>true</gravity>
     <self_collide>false</self_collide>
-    <material value="Gazebo/Blue" />
+    <!--material value="Gazebo/Blue" /-->
   </gazebo>
   <gazebo reference="${arm_id}_link5">
