Commit message: Decoupled separator distancer and separator base

File: schunk_lwa4p_description/urdf/lwa4p/lwa4p_arm_hand_powerline.urdf.xacro (robot description, xacro)
@@ -10,4 +10,7 @@
   </xacro:include>
   <xacro:include filename="$(find schunk_lwa4p_description)/urdf/powerline.xacro" >
+	<xacro:arg name="gazebo" value="${gazebo}"/>
+  </xacro:include>
+  <xacro:include filename="$(find schunk_lwa4p_description)/urdf/separator_distancer.xacro" >
 	<xacro:arg name="gazebo" value="${gazebo}"/>
   </xacro:include>
@@ -40,4 +43,6 @@
   <!-- tool -->
   <xacro:separator ns="lwa4p" rpy="0 0 ${-pi/4}" connected_to="lwa4p_link6" safety_distance="0.03"/>
+  <!-- distancer -->
+  <xacro:separator_distancer ns="lwa4p" rpy="0 0 0" xyz="0 0 0"/>
   <!-- powerline -->
   <xacro:powerline base_x="0" base_y="0" base_z="0.25" x_distance="0.5" y_distance="1.25" gazebo="true" two_cables="true" cable_distance="0.3"/>

File: schunk_lwa4p_description/urdf/lwa4p/lwa4p_arm_separator_powerline.urdf.xacro (robot description, xacro)
@@ -7,4 +7,7 @@
   </xacro:include>
   <xacro:include filename="$(find schunk_lwa4p_description)/urdf/tools/separator.xacro">
+	<xacro:arg name="gazebo" value="${gazebo}"/>
+  </xacro:include>
+  <xacro:include filename="$(find schunk_lwa4p_description)/urdf/tools/separator_distancer.xacro">
 	<xacro:arg name="gazebo" value="${gazebo}"/>
   </xacro:include>
@@ -38,4 +41,6 @@
   <!-- tool -->
   <xacro:separator ns="lwa4p" rpy="0 0 0" connected_to="lwa4p_link6" safety_distance="0.03"/>
+  <!-- distancer -->
+  <!--xacro:separator_distancer ns="lwa4p" rpy="0 0 0" xyz="0 0 0.05"/-->
   <!-- powerline -->
   <xacro:powerline base_x="0" base_y="0" base_z="0.25" x_distance="0.5" y_distance="1.25" gazebo="true" two_cables="true" cable_distance="0.3"/>

File: schunk_lwa4p_description/urdf/tools/separator_distancer.urdf.xacro (robot description, xacro)
@@ -1,4 +1,4 @@
 <?xml version="1.0" encoding="utf-8"?>
-<robot xmlns:xacro="http://www.ros.org/wiki/xacro" name="hand">
+<robot xmlns:xacro="http://www.ros.org/wiki/xacro" name="separator_distancer">
     <xacro:include filename="separator_distancer.xacro"/>
 </robot>

File: schunk_lwa4p_description/urdf/tools/separator_distancer.xacro (robot description, xacro)
@@ -1,5 +1,5 @@
 <?xml version="1.0" encoding="utf-8"?>
 <robot xmlns:xacro="http://www.ros.org/wiki/xacro" name="separator_distancer">
-    <xacro:macro name="separator_distancer" params="rpy:='0 0 0' ns:='' xyz:='0 0 0.1'">
+    <xacro:macro name="separator_distancer" params="rpy:='0 0 0' ns:='' xyz:='2 2 0.1'">
         <xacro:property name="scale_factor" value="3.937007"/>
         <xacro:arg name="gazebo" default="true"/>
@@ -8,4 +8,9 @@
             <xacro:include filename="$(find schunk_lwa4p_description)/urdf/tools/separator_distancer.gazebo.xacro"/>
         </xacro:if>
+        <!--joint name="separator_distancer_joint" type="floating" />
+            <origin xyz="0 0 0" rpy="0 0 0"/>
+            <parent link="separator_base"/>
+            <child link="spearator_main"/>
+        </joint-->
         <link name="separator_main">
             <inertial>
@@ -28,6 +33,6 @@
             </collision>
         </link>
-        <joint name="world_separator" type="floating">
-            <parent link="world"/>
+        <joint name="world_separator" type="fixed">
+            <parent link="separator_base"/>
             <child link="separator_main"/>
             <origin rpy="${rpy}" xyz="${xyz}"/>
