Commit message: Separator decoupling (still)

File: schunk_lwa4p_description/urdf/lwa4p/lwa4p_arm_separator.urdf.xacro (robot description, xacro)
@@ -46,4 +46,4 @@
   <xacro:separator ns="lwa4p" rpy="0 0 0" connected_to="lwa4p_link6" safety_distance="0.03"/>
   <!-- separator distancer -->
-  <xacro:separator_distancer ns="lwa4p" rpy="0 0 0" xyz="0 0 1.5"/>
+  <xacro:separator_distancer ns="lwa4p" rpy="0 0 0" xyz="0 0 0.05"/>
 </robot>

File: schunk_lwa4p_description/urdf/tools/separator_distancer.xacro (robot description, xacro)
@@ -1,5 +1,5 @@
 <?xml version="1.0" encoding="utf-8"?>
 <robot xmlns:xacro="http://www.ros.org/wiki/xacro" name="separator_distancer">
-    <xacro:macro name="separator_distancer" params="rpy:='0 0 0' ns:='' xyz:='2 2 0.1'">
+    <xacro:macro name="separator_distancer" params="rpy:='0 0 0' ns:='' xyz:='0 0 0.01' ">
         <xacro:property name="scale_factor" value="3.937007"/>
         <xacro:arg name="gazebo" default="true"/>
@@ -8,9 +8,10 @@
             <xacro:include filename="$(find schunk_lwa4p_description)/urdf/tools/separator_distancer.gazebo.xacro"/>
         </xacro:if>
-        <!--joint name="separator_distancer_joint" type="floating" />
-            <origin xyz="0 0 0" rpy="0 0 0"/>
+        <joint name="separator_distancer_joint" type="fixed" >
+            <origin xyz="${xyz}" rpy="${rpy}"/>
+            <!--parent link="lwa4p_link6"/-->
             <parent link="separator_base"/>
-            <child link="spearator_main"/>
-        </joint-->
+            <child link="separator_main"/>
+        </joint>
         <link name="separator_main">
             <inertial>
@@ -33,9 +34,4 @@
             </collision>
         </link>
-        <joint name="world_separator" type="fixed">
-            <parent link="separator_base"/>
-            <child link="separator_main"/>
-            <origin rpy="${rpy}" xyz="${xyz}"/>
-        </joint>
         <link name="separator_right_head">
             <inertial>

Commit message: Updated README.md
Added some stuff for FastIK and some stuff for Descartes planning

Removed mistake

Removed vscode core mistake

File: schunk_lwa4p_description/urdf/lwa4p/lwa4p_arm_separator.urdf.xacro (robot description, xacro)
@@ -41,5 +41,5 @@
   <!-- arm -->
   <xacro:lwa4p_arm arm_id="lwa4p" parent="base_link" has_podest="true" >
-    <origin xyz="0 0 0.50" rpy="0 0 0" />
+    <origin xyz="0 0 0.25" rpy="0 0 0" />
   </xacro:lwa4p_arm>
   <!-- tool -->

Commit message: Added some updates to enable inverse kinematics for melodic

File: schunk_lwa4p_description/urdf/lwa4p/lwa4p_arm_separator.urdf.xacro (robot description, xacro)
@@ -41,5 +41,5 @@
   <!-- arm -->
   <xacro:lwa4p_arm arm_id="lwa4p" parent="base_link" has_podest="true" >
-    <origin xyz="0 0 0.25" rpy="0 0 0" />
+    <origin xyz="0 0 0.5" rpy="0 0 0" />
   </xacro:lwa4p_arm>
   <!-- tool -->
