Commit message: Added separator controllers

File: schunk_lwa4p_description/urdf/lwa4p/lwa4p_arm.gazebo.xacro (robot description, xacro)
@@ -11,5 +11,5 @@
     <gravity>true</gravity>
       <self_collide>false</self_collide>
-      <material value="Gazebo/LightGrey" />
+      <material value="Gazebo/Grey" />
   </gazebo>
   <gazebo reference="${arm_id}_link2">
@@ -21,5 +21,5 @@
     <gravity>true</gravity>
     <self_collide>false</self_collide>
-    <material value="Gazebo/LightGrey" />
+    <material value="Gazebo/Grey" />
   </gazebo>
   <gazebo reference="${arm_id}_link4">
@@ -31,5 +31,5 @@
     <gravity>true</gravity>
     <self_collide>false</self_collide>
-    <material value="Gazebo/LightGrey" />
+    <material value="Gazebo/Grey" />
   </gazebo>
   <gazebo reference="${arm_id}_link6">
@@ -37,9 +37,4 @@
     <self_collide>false</self_collide>
     <material value="Gazebo/Blue" />
-  </gazebo>
-  <gazebo reference="${arm_id}_link7">
-    <gravity>true</gravity>
-    <self_collide>false</self_collide>
-    <material value="Gazebo/LightGrey" />
   </gazebo>
   <transmission name="${arm_id}_joint1_trans">

File: schunk_lwa4p_description/urdf/lwa4p/lwa4p_arm.xacro (robot description, xacro)
@@ -64,5 +64,5 @@
           <mesh filename="package://schunk_lwa4p_description/meshes/lwa4p/stl/arm_1_link.stl" />
         </geometry>
-        <!--material name="Schunk/Blue" /-->
+        <material name="Schunk/Blue" />
       </visual>
       <collision>
@@ -96,5 +96,5 @@
           <mesh filename="package://schunk_lwa4p_description/meshes/lwa4p/stl/arm_2_link.stl" />
         </geometry>
-        <!--material name="Schunk/LightGrey" /-->
+        <material name="Schunk/LightGrey" />
       </visual>
       <collision>
@@ -129,5 +129,5 @@
           <mesh filename="package://schunk_lwa4p_description/meshes/lwa4p/stl/arm_3_link.stl" />
         </geometry>
-        <!--material name="Schunk/LightGrey" /-->
+        <material name="Schunk/LightGrey" />
       </visual>
       <collision>
@@ -162,5 +162,5 @@
           <mesh filename="package://schunk_lwa4p_description/meshes/lwa4p/stl/arm_4_link.stl" />
         </geometry>
-        <!--material name="Schunk/LightGrey" /-->
+        <material name="Schunk/LightGrey" />
       </visual>
       <collision>
@@ -195,5 +195,5 @@
           <mesh filename="package://schunk_lwa4p_description/meshes/lwa4p/stl/arm_5_link.stl" />
         </geometry>
-        <!--material name="Schunk/Blue" /-->
+        <material name="Schunk/Blue" />
       </visual>
       <collision>
@@ -228,5 +228,5 @@
           <mesh filename="package://schunk_lwa4p_description/meshes/lwa4p/stl/arm_6_link.stl" />
         </geometry>
-        <!--material name="Schunk/LightGrey" /-->
+        <material name="Schunk/LightGrey" />
       </visual>
       <collision>

File: schunk_lwa4p_description/urdf/lwa4p/lwa4p_arm_separator.gazebo.xacro (robot description, xacro)
@@ -38,33 +38,28 @@
     <material value="Gazebo/Blue" />
   </gazebo>
-  <gazebo reference="${arm_id}_link7">
-    <gravity>true</gravity>
-    <self_collide>false</self_collide>
-    <material value="Gazebo/LightGrey" />
+  <gazebo reference="separator_base">
+    <material value="Gazebo/Red" />
   </gazebo>
-  <gazebo reference="separator_base">
-        <material value="Gazebo/Red " />
-    </gazebo>
-    <gazebo reference="separator_main">
-        <material value="Gazebo/ZincYellow" />
-    </gazebo>
-    <gazebo reference="separator_right_back_holder">
-        <material value="Gazebo/Green" />
-    </gazebo>
-    <gazebo reference="separator_right_front_holder">
-        <material value="Gazebo/Green" />
-    </gazebo>
-    <gazebo reference="separator_right_front_holder">
-        <material value="Gazebo/Green" />
-    </gazebo>
-    <gazebo reference="separator_left_front_holder">
-        <material value="Gazebo/Green" />
-    </gazebo>
-    <gazebo reference="separator_right_head">
-        <material value="Gazebo/YellowGlow" />
-    </gazebo>
-    <gazebo reference="separator_left_head">
-        <material value="Gazebo/YellowGlow" />
-    </gazebo>
+  <gazebo reference="separator_main">
+    <material value="Gazebo/ZincYellow" />
+  </gazebo>
+  <gazebo reference="separator_right_back_holder">
+    <material value="Gazebo/Green" />
+  </gazebo>
+  <gazebo reference="separator_right_front_holder">
+    <material value="Gazebo/Green" />
+  </gazebo>
+  <gazebo reference="separator_right_front_holder">
+    <material value="Gazebo/Green" />
+  </gazebo>
+  <gazebo reference="separator_left_front_holder">
+    <material value="Gazebo/Green" />
+  </gazebo>
+  <gazebo reference="separator_right_head">
+    <material value="Gazebo/YellowGlow" />
+  </gazebo>
+  <gazebo reference="separator_left_head">
+    <material value="Gazebo/YellowGlow" />
+  </gazebo>
   <transmission name="${arm_id}_joint1_trans">
     <type>transmission_interface/SimpleTransmission</type>

File: schunk_lwa4p_description/urdf/tools/separator.gazebo.xacro (robot description, xacro)
@@ -5,4 +5,5 @@
     </gazebo>
     <gazebo reference="separator_main">
+        <gravity>false</gravity>
         <material value="Gazebo/ZincYellow" />
     </gazebo>
@@ -26,5 +27,5 @@
     </gazebo>
     <transmission name="separator_base_main_trans">
-    <type>transmission_interface/SimpleTransmission</type>
+        <type>transmission_interface/SimpleTransmission</type>
         <joint name="separator_base_main_joint">
             <hardwareInterface>hardware_interface/PositionJointInterface</hardwareInterface>
@@ -51,4 +52,40 @@
             <mechanicalReduction>1</mechanicalReduction>
         </actuator>
-    </transmission>s
+    </transmission>
+    <transmission name="separator_right_front_trans">
+        <type>transmission_interface/SimpleTransmission</type>
+        <joint name="separator_right_front_joint">
+            <hardwareInterface>hardware_interface/PositionJointInterface</hardwareInterface>
+        </joint>
+        <actuator name="separator_right_front_joint_motor">
+            <mechanicalReduction>1</mechanicalReduction>
+        </actuator>
+    </transmission>
+    <transmission name="separator_right_back_trans">
+        <type>transmission_interface/SimpleTransmission</type>
+        <joint name="separator_right_back_joint">
+            <hardwareInterface>hardware_interface/PositionJointInterface</hardwareInterface>
+        </joint>
+        <actuator name="separator_right_back_joint_motor">
+            <mechanicalReduction>1</mechanicalReduction>
+        </actuator>
+    </transmission>
+    <transmission name="separator_left_front_trans">
+        <type>transmission_interface/SimpleTransmission</type>
+        <joint name="separator_left_front_joint">
+            <hardwareInterface>hardware_interface/PositionJointInterface</hardwareInterface>
+        </joint>
+        <actuator name="separator_left_front_joint_motor">
+            <mechanicalReduction>1</mechanicalReduction>
+        </actuator>
+    </transmission>
+    <transmission name="separator_left_back_trans">
+        <type>transmission_interface/SimpleTransmission</type>
+        <joint name="separator_left_back_joint">
+            <hardwareInterface>hardware_interface/PositionJointInterface</hardwareInterface>
+        </joint>
+        <actuator name="separator_left_back_joint_motor">
+            <mechanicalReduction>1</mechanicalReduction>
+        </actuator>
+    </transmission>
 </robot>

File: schunk_lwa4p_description/urdf/tools/separator.xacro (robot description, xacro)
@@ -12,5 +12,5 @@
             <xacro:if value="$(arg gazebo)">
             <!-- Gazebo Tags -->
-            <xacro:include filename="$(find schunk_lwa4p_moveit)/urdf/tools/separator.gazebo.xacro"/>
+            <xacro:include filename="$(find schunk_lwa4p_description)/urdf/tools/separator.gazebo.xacro"/>
         </xacro:if>
         <xacro:property name="scale_factor" value="3.937007"/>
@@ -33,5 +33,5 @@
                 <origin rpy="0 0 0" xyz="0 0 0"/>
                 <geometry>
-                    <mesh filename="package://schunk_lwa4p_moveit/meshes/separator/baza2.STL" scale="0.0254 0.0254 0.0254"/>
+                    <mesh filename="package://schunk_lwa4p_description/meshes/separator/baza2.STL" scale="0.0254 0.0254 0.0254"/>
                 </geometry>
                 <material name="blue"/>
@@ -40,5 +40,5 @@
                 <origin rpy="0 0 0" xyz="0 0 0"/>
                 <geometry>
-                    <mesh filename="package://schunk_lwa4p_moveit/meshes/separator/baza2.STL" scale="0.0254 0.0254 0.0254"/>
+                    <mesh filename="package://schunk_lwa4p_description/meshes/separator/baza2.STL" scale="0.0254 0.0254 0.0254"/>
                 </geometry>
             </collision>
@@ -53,5 +53,5 @@
                 <origin rpy="0 0 0" xyz="0 0 0"/>
                 <geometry>
-                    <mesh filename="package://schunk_lwa4p_moveit/meshes/separator/separator3.STL" scale="0.0254 0.0254 0.0254"/>
+                    <mesh filename="package://schunk_lwa4p_description/meshes/separator/separator3.STL" scale="0.0254 0.0254 0.0254"/>
                 </geometry>
                 <material name="white"/>
@@ -60,5 +60,5 @@
                 <origin rpy="0 0 0" xyz="0 0 0"/>
                 <geometry>
-                    <mesh filename="package://schunk_lwa4p_moveit/meshes/separator/separator3.STL" scale="0.0254 0.0254 0.0254"/>
+                    <mesh filename="package://schunk_lwa4p_description/meshes/separator/separator3.STL" scale="0.0254 0.0254 0.0254"/>
                 </geometry>
             </collision>
@@ -67,6 +67,7 @@
             <parent link="separator_base"/>
             <child link="separator_main"/>
-            <origin xyz="0 0 ${0.19685/scale_factor}" rpy="0 0 0"/>
-            <limit effort="1000" velocity="0.05" lower="-0.5" upper="0.5"/>
+            <!-- Here is BUG FIX FOR SEPARATOR MAIN, at loading somehow Gazebo forgots to take podest into consideration -->
+            <origin xyz="0 0 ${0.19685/scale_factor + 0.5}" rpy="0 0 0"/>
+            <limit effort="1000" velocity="0.00" lower="-0.5" upper="0.5"/>
             <axis xyz="0 0 1"/>
         </joint>
@@ -80,5 +81,5 @@
                 <origin rpy="0 0 0" xyz="-${0.032/scale_factor} -${0.385443/scale_factor} -${0.16/scale_factor}"/>
                 <geometry>
-                    <mesh filename="package://schunk_lwa4p_moveit/meshes/separator/desni_prednji_drzac.STL" scale="0.0254 0.0254 0.0254"/>
+                    <mesh filename="package://schunk_lwa4p_description/meshes/separator/desni_prednji_drzac.STL" scale="0.0254 0.0254 0.0254"/>
                 </geometry>
             </visual>
@@ -86,5 +87,5 @@
                 <origin rpy="0 0 0" xyz="-${0.032/scale_factor} -${0.385443/scale_factor} -${0.16/scale_factor}"/>
                 <geometry>
-                    <mesh filename="package://schunk_lwa4p_moveit/meshes/separator/desni_prednji_drzac.STL" scale="0.0254 0.0254 0.0254"/>
+                    <mesh filename="package://schunk_lwa4p_description/meshes/separator/desni_prednji_drzac.STL" scale="0.0254 0.0254 0.0254"/>
                 </geometry>
             </collision>
@@ -106,5 +107,5 @@
                 <origin rpy="0 0 0" xyz="-${0.032/scale_factor} ${0.385443/scale_factor} -${0.16/scale_factor}"/>
                 <geometry>
-                    <mesh filename="package://schunk_lwa4p_moveit/meshes/separator/desni_zadnji_drzac.STL" scale="0.0254 0.0254 0.0254"/>
+                    <mesh filename="package://schunk_lwa4p_description/meshes/separator/desni_zadnji_drzac.STL" scale="0.0254 0.0254 0.0254"/>
                 </geometry>
             </visual>
@@ -112,5 +113,5 @@
                 <origin rpy="0 0 0" xyz="-${0.032/scale_factor} ${0.385443/scale_factor} -${0.16/scale_factor}"/>
                 <geometry>
-                    <mesh filename="package://schunk_lwa4p_moveit/meshes/separator/desni_zadnji_drzac.STL" scale="0.0254 0.0254 0.0254"/>
+                    <mesh filename="package://schunk_lwa4p_description/meshes/separator/desni_zadnji_drzac.STL" scale="0.0254 0.0254 0.0254"/>
                 </geometry>
             </collision>
@@ -132,5 +133,5 @@
                 <origin rpy="0 0 0" xyz="${0.032/scale_factor} -${0.385443/scale_factor} -${0.16/scale_factor}"/>
                 <geometry>
-                    <mesh filename="package://schunk_lwa4p_moveit/meshes/separator/lijevi_prednji_drzac.STL" scale="0.0254 0.0254 0.0254"/>
+                    <mesh filename="package://schunk_lwa4p_description/meshes/separator/lijevi_prednji_drzac.STL" scale="0.0254 0.0254 0.0254"/>
                 </geometry>
             </visual>
@@ -138,5 +139,5 @@
                 <origin rpy="0 0 0" xyz="${0.032/scale_factor} -${0.385443/scale_factor} -${0.16/scale_factor}"/>
                 <geometry>
-                    <mesh filename="package://schunk_lwa4p_moveit/meshes/separator/lijevi_prednji_drzac.STL" scale="0.0254 0.0254 0.0254"/>
+                    <mesh filename="package://schunk_lwa4p_description/meshes/separator/lijevi_prednji_drzac.STL" scale="0.0254 0.0254 0.0254"/>
                 </geometry>
             </collision>
@@ -158,5 +159,5 @@
                 <origin rpy="0 0 0" xyz="${0.032/scale_factor} ${0.385443/scale_factor}  -${0.16/scale_factor}"/>
                 <geometry>
-                    <mesh filename="package://schunk_lwa4p_moveit/meshes/separator/lijevi_zadnji_drzac.STL" scale="0.0254 0.0254 0.0254"/>
+                    <mesh filename="package://schunk_lwa4p_description/meshes/separator/lijevi_zadnji_drzac.STL" scale="0.0254 0.0254 0.0254"/>
                 </geometry>
             </visual>
@@ -164,5 +165,5 @@
                 <origin rpy="0 0 0" xyz="${0.032/scale_factor} ${0.385443/scale_factor} -${0.16/scale_factor}"/>
                 <geometry>
-                    <mesh filename="package://schunk_lwa4p_moveit/meshes/separator/lijevi_zadnji_drzac.STL" scale="0.0254 0.0254 0.0254"/>
+                    <mesh filename="package://schunk_lwa4p_description/meshes/separator/lijevi_zadnji_drzac.STL" scale="0.0254 0.0254 0.0254"/>
                 </geometry>
             </collision>
@@ -184,5 +185,5 @@
                 <origin rpy="0 0 0" xyz="0 ${0.545/scale_factor} -0.01"/>
                 <geometry>
-                    <mesh filename="package://schunk_lwa4p_moveit/meshes/separator/separator1.STL" scale="0.0254 0.0254 0.0254"/>
+                    <mesh filename="package://schunk_lwa4p_description/meshes/separator/separator1.STL" scale="0.0254 0.0254 0.0254"/>
                 </geometry>
                 <material name="custom"/>
@@ -191,5 +192,5 @@
                 <origin rpy="0 0 0" xyz="0 ${0.545/scale_factor} -0.01"/>
                 <geometry>
-                    <mesh filename="package://schunk_lwa4p_moveit/meshes/separator/separator1.STL" scale="0.0254 0.0254 0.0254"/>
+                    <mesh filename="package://schunk_lwa4p_description/meshes/separator/separator1.STL" scale="0.0254 0.0254 0.0254"/>
                 </geometry>
             </collision>
@@ -212,5 +213,5 @@
                 <origin rpy="0 0 0" xyz="0 -${0.545/scale_factor} -0.01"/>
                 <geometry>
-                    <mesh filename="package://schunk_lwa4p_moveit/meshes/separator/separator2.STL" scale="0.0254 0.0254 0.0254"/>
+                    <mesh filename="package://schunk_lwa4p_description/meshes/separator/separator2.STL" scale="0.0254 0.0254 0.0254"/>
                 </geometry>
                 <material name="custom"/>
@@ -219,5 +220,5 @@
                 <origin rpy="0 0 0" xyz="0 -${0.545/scale_factor} -0.01"/>
                 <geometry>
-                    <mesh filename="package://schunk_lwa4p_moveit/meshes/separator/separator2.STL" scale="0.0254 0.0254 0.0254"/>
+                    <mesh filename="package://schunk_lwa4p_description/meshes/separator/separator2.STL" scale="0.0254 0.0254 0.0254"/>
                 </geometry>
             </collision>
