Commit message: Decoupled separator tool and distancer

File: schunk_lwa4p_description/urdf/lwa4p/lwa4p_arm.gazebo.xacro (robot description, xacro)
@@ -2,10 +2,4 @@
 <robot xmlns:xacro="http://www.ros.org/wiki/xacro" name="lwa4p">
   <xacro:include filename="$(find schunk_lwa4p_description)/urdf/materials.urdf.xacro"/>
-  <gazebo>
-    <plugin name="gazebo_ros_control" filename="libgazebo_ros_control.so">
-      <robotNamespace>/lwa4p</robotNamespace>
-      <legacyModeNS>true</legacyModeNS>
-    </plugin>
-  </gazebo>
   <gazebo reference="${arm_id}_link1">
     <gravity>true</gravity>
@@ -37,4 +31,19 @@
     <self_collide>false</self_collide>
     <material value="Gazebo/Blue" />
+  </gazebo>
+  <!-- To have fully consistent Gazebo simulation it should have 2 IMUs for 1 power cable and 3 IMUs for 2 power cables -->
+  <!--xacro:if value=$(arg init_imu)>
+      <gazebo>
+      <plugin name="gazebo_ros_control" filename="libgazebo_ros_magnetometer.so">
+        <robotNamespace>/lwa4p</robotNamespace>
+        <legacyModeNS>true</legacyModeNS>
+      </plugin>
+    </gazebo>
+  </xacro:if-->
+  <gazebo>
+    <plugin name="gazebo_ros_control" filename="libgazebo_ros_control.so">
+      <robotNamespace>/lwa4p</robotNamespace>
+      <legacyModeNS>true</legacyModeNS>
+    </plugin>
   </gazebo>
   <transmission name="${arm_id}_joint1_trans">

File: schunk_lwa4p_description/urdf/lwa4p/lwa4p_arm_separator.urdf.xacro (robot description, xacro)
@@ -7,4 +7,7 @@
   </xacro:include>
   <xacro:include filename="$(find schunk_lwa4p_description)/urdf/tools/separator.xacro" >
+	<xacro:arg name="gazebo" value="${gazebo}"/>
+  </xacro:include>
+  <xacro:include filename="$(find schunk_lwa4p_description)/urdf/tools/separator_distancer.xacro" >
 	<xacro:arg name="gazebo" value="${gazebo}"/>
   </xacro:include>
@@ -42,3 +45,5 @@
   <!-- tool -->
   <xacro:separator ns="lwa4p" rpy="0 0 0" connected_to="lwa4p_link6" safety_distance="0.03"/>
+  <!-- separator distancer -->
+  <xacro:separator_distancer ns="lwa4p" rpy="0 0 0" xyz="0 0 1.5"/>
 </robot>

File: schunk_lwa4p_description/urdf/powerline.xacro (robot description, xacro)
@@ -24,5 +24,5 @@
 		        <origin xyz="0 0 0" rpy="0 0 0" />
 		        <geometry>
-		            <cylinder radius="0.05" length="0.75"/>
+		            <cylinder radius="0.1" length="0.75"/>
 		        </geometry>
 		    </collision>
@@ -33,5 +33,5 @@
 		    </inertial>
 	    </link>
-        <joint name="base_powerline_link2" type="fixed">
+        <joint name="base_powerline_link2"  type="fixed">
             <origin xyz="${x_distance} ${y_distance} 0.375" rpy="0 0 0"/>
             <parent link="base_link"/>

File: schunk_lwa4p_description/urdf/tools/separator.gazebo.xacro (robot description, xacro)
@@ -3,8 +3,4 @@
     <gazebo reference="separator_base">
         <material value="Gazebo/Red " />
-    </gazebo>
-    <gazebo reference="separator_main">
-        <gravity>false</gravity>
-        <material value="Gazebo/ZincYellow" />
     </gazebo>
     <gazebo reference="separator_right_back_holder">
@@ -20,37 +16,4 @@
         <material value="Gazebo/Green" />
     </gazebo>
-    <gazebo reference="separator_right_head">
-        <material value="Gazebo/YellowGlow" />
-    </gazebo>
-    <gazebo reference="separator_left_head">
-        <material value="Gazebo/YellowGlow" />
-    </gazebo>
-    <transmission name="separator_base_main_trans">
-        <type>transmission_interface/SimpleTransmission</type>
-        <joint name="separator_base_main_joint">
-            <hardwareInterface>hardware_interface/PositionJointInterface</hardwareInterface>
-        </joint>
-        <actuator name="separator_base_main_joint_motor">
-            <mechanicalReduction>1</mechanicalReduction>
-        </actuator>
-    </transmission>
-    <transmission name="separator_right_head_trans">
-        <type>transmission_interface/SimpleTransmission</type>
-        <joint name="separator_main_right_head_joint">
-            <hardwareInterface>hardware_interface/PositionJointInterface</hardwareInterface>
-        </joint>
-        <actuator name="separator_main_right_head_joint_motor">
-            <mechanicalReduction>1</mechanicalReduction>
-        </actuator>
-    </transmission>
-    <transmission name="separator_left_head_trans">
-        <type>transmission_interface/SimpleTransmission</type>
-        <joint name="separator_main_left_head_joint">
-            <hardwareInterface>hardware_interface/PositionJointInterface</hardwareInterface>
-        </joint>
-        <actuator name="separator_main_left_head_joint_motor">
-            <mechanicalReduction>1</mechanicalReduction>
-        </actuator>
-    </transmission>
     <transmission name="separator_right_front_trans">
         <type>transmission_interface/SimpleTransmission</type>

File: schunk_lwa4p_description/urdf/tools/separator.xacro (robot description, xacro)
@@ -44,32 +44,4 @@
             </collision>
         </link>
-        <link name="separator_main">
-            <inertial>
-                <origin rpy="0 0 0" xyz="0 0 0"/>
-                <mass value="1" />
-                <inertia ixx="1" ixy="0.0" ixz="0.0" iyy="1" iyz="0.0" izz="1"/>
-            </inertial>
-            <visual>
-                <origin rpy="0 0 0" xyz="0 0 0"/>
-                <geometry>
-                    <mesh filename="package://schunk_lwa4p_description/meshes/separator/separator3.STL" scale="0.0254 0.0254 0.0254"/>
-                </geometry>
-                <material name="white"/>
-            </visual>
-            <collision>
-                <origin rpy="0 0 0" xyz="0 0 0"/>
-                <geometry>
-                    <mesh filename="package://schunk_lwa4p_description/meshes/separator/separator3.STL" scale="0.0254 0.0254 0.0254"/>
-                </geometry>
-            </collision>
-        </link>
-        <joint name="separator_base_main_joint" type="prismatic">
-            <parent link="separator_base"/>
-            <child link="separator_main"/>
-            <!-- Here is BUG FIX FOR SEPARATOR MAIN, at loading somehow Gazebo forgots to take podest into consideration -->
-            <origin xyz="0 0 ${0.19685/scale_factor + 0.5}" rpy="0 0 0"/>
-            <limit effort="1000" velocity="0.00" lower="-0.5" upper="0.5"/>
-            <axis xyz="0 0 1"/>
-        </joint>
         <link name="right_front_holder">
             <inertial>
@@ -176,59 +148,4 @@
             <axis xyz="0 1 0"/>
         </joint>
-        <link name="separator_right_head">
-            <inertial>
-                <origin rpy="0 0 0" xyz="0 0 0"/>
-                <mass value="0.2" />
-                <inertia ixx="1" ixy="0.0" ixz="0.0" iyy="1" iyz="0.0" izz="1"/>
-            </inertial>
-            <visual>
-                <origin rpy="0 0 0" xyz="0 ${0.545/scale_factor} -0.01"/>
-                <geometry>
-                    <mesh filename="package://schunk_lwa4p_description/meshes/separator/separator1.STL" scale="0.0254 0.0254 0.0254"/>
-                </geometry>
-                <material name="custom"/>
-            </visual>
-            <collision>
-                <origin rpy="0 0 0" xyz="0 ${0.545/scale_factor} -0.01"/>
-                <geometry>
-                    <mesh filename="package://schunk_lwa4p_description/meshes/separator/separator1.STL" scale="0.0254 0.0254 0.0254"/>
-                </geometry>
-            </collision>
-        </link>
-        <joint name="separator_main_right_head_joint" type="revolute">
-            <parent link="separator_main"/>
-            <child link="separator_right_head"/>
-            <origin xyz="0 -${0.54/scale_factor} 0" rpy="0 0 0"/>
-            <limit effort="10" velocity="0.5" lower="-0.45" upper="0"/>
-            <axis xyz="1 0 0"/>
-        </joint>
-        <link name="separator_left_head">
-            <inertial>
-                <origin rpy="0 0 0" xyz="0 0 0"/>
-                <mass value="0.2" />
-                <inertia ixx="1" ixy="0.0" ixz="0.0" iyy="1" iyz="0.0" izz="1"/>
-                <material name="white"/>
-            </inertial>
-            <visual>
-                <origin rpy="0 0 0" xyz="0 -${0.545/scale_factor} -0.01"/>
-                <geometry>
-                    <mesh filename="package://schunk_lwa4p_description/meshes/separator/separator2.STL" scale="0.0254 0.0254 0.0254"/>
-                </geometry>
-                <material name="custom"/>
-            </visual>
-            <collision>
-                <origin rpy="0 0 0" xyz="0 -${0.545/scale_factor} -0.01"/>
-                <geometry>
-                    <mesh filename="package://schunk_lwa4p_description/meshes/separator/separator2.STL" scale="0.0254 0.0254 0.0254"/>
-                </geometry>
-            </collision>
-        </link>
-        <joint name="separator_main_left_head_joint" type="revolute">
-            <parent link="separator_main"/>
-            <child link="separator_left_head"/>
-            <origin xyz="0 ${0.54/scale_factor} 0" rpy="0 0 0"/>
-            <limit effort="10" velocity="0.5" lower="0" upper="0.45"/>
-            <axis xyz="1 0 0"/>
-        </joint>
     </xacro:macro>
 </robot>

Commit message: Added initial velocity controls and server updates

File: schunk_lwa4p_description/urdf/lwa4p/lwa4p_arm.gazebo.xacro (robot description, xacro)
@@ -51,5 +51,5 @@
     <joint name="${arm_id}_joint1">
       <hardwareInterface>hardware_interface/PositionJointInterface</hardwareInterface>
-      <!--hardwareInterface>hardware_interface/VelocityJointInterface</hardwareInterface-->
+      <!--hardwareInterface>hardware_interface/VelocityJointInterface</hardwareInterface!-->
     </joint>
     <actuator name="${arm_id}_joint1_motor">
@@ -61,5 +61,6 @@
     <joint name="${arm_id}_joint2">
       <hardwareInterface>hardware_interface/PositionJointInterface</hardwareInterface>
-      <!--hardwareInterface>hardware_interface/VelocityJointInterface</hardwareInterface-->    </joint>
+      <!--hardwareInterface>hardware_interface/VelocityJointInterface</hardwareInterface!-->
+    </joint>
     <actuator name="${arm_id}_joint2_motor">
       <mechanicalReduction>1</mechanicalReduction>
@@ -70,5 +71,5 @@
     <joint name="${arm_id}_joint3">
       <hardwareInterface>hardware_interface/PositionJointInterface</hardwareInterface>
-      <!--hardwareInterface>hardware_interface/VelocityJointInterface</hardwareInterface-->
+      <!--hardwareInterface>hardware_interface/VelocityJointInterface</hardwareInterface!-->
     </joint>
     <actuator name="${arm_id}_joint3_motor">
@@ -80,5 +81,5 @@
     <joint name="${arm_id}_joint4">
       <hardwareInterface>hardware_interface/PositionJointInterface</hardwareInterface>
-      <!--hardwareInterface>hardware_interface/VelocityJointInterface</hardwareInterface-->
+      <!--hardwareInterface>hardware_interface/VelocityJointInterface</hardwareInterface!-->
     </joint>
     <actuator name="${arm_id}_joint4_motor">
@@ -90,5 +91,5 @@
     <joint name="${arm_id}_joint5">
       <hardwareInterface>hardware_interface/PositionJointInterface</hardwareInterface>
-      <!--hardwareInterface>hardware_interface/VelocityJointInterface</hardwareInterface-->
+      <!--hardwareInterface>hardware_interface/VelocityJointInterface</hardwareInterface!-->
     </joint>
     <actuator name="${arm_id}_joint5_motor">
@@ -100,5 +101,5 @@
     <joint name="${arm_id}_joint6">
       <hardwareInterface>hardware_interface/PositionJointInterface</hardwareInterface>
-      <!--hardwareInterface>hardware_interface/VelocityJointInterface</hardwareInterface-->
+      <!--hardwareInterface>hardware_interface/VelocityJointInterface</hardwareInterface!-->
     </joint>
     <actuator name="${arm_id}_joint6_motor">

File: schunk_lwa4p_description/urdf/lwa4p/lwa4p_arm_separator.gazebo.xacro (robot description, xacro)
@@ -76,5 +76,6 @@
     <joint name="${arm_id}_joint2">
       <hardwareInterface>hardware_interface/PositionJointInterface</hardwareInterface>
-      <!--hardwareInterface>hardware_interface/VelocityJointInterface</hardwareInterface-->    </joint>
+      <!--hardwareInterface>hardware_interface/VelocityJointInterface</hardwareInterface-->
+    </joint>
     <actuator name="${arm_id}_joint2_motor">
       <mechanicalReduction>1</mechanicalReduction>
