Commit message: Added parametrized powerline model

File: schunk_lwa4p_description/urdf/lwa4p/lwa4p_arm_separator_powerline.urdf.xacro (robot description, xacro)
@@ -41,7 +41,7 @@
   <!-- tool -->
   <xacro:separator ns="lwa4p" rpy="0 0 0" connected_to="lwa4p_link6" safety_distance="0.03"/>
-  <!-- distancer -->
-  <!--xacro:separator_distancer ns="lwa4p" rpy="0 0 0" xyz="0 0 0.05"/-->
+  <!-- separator distancer -->
+  <xacro:separator_distancer ns="lwa4p" rpy="0 0 0" xyz="0 0 0.05"/>
   <!-- powerline -->
-  <xacro:powerline base_x="0" base_y="0" base_z="0.25" x_distance="0.5" y_distance="1.25" gazebo="true" two_cables="true" cable_distance="0.3"/>
+  <xacro:powerline base_x="0" base_y="0" powerline_height="1.0" x_distance="0.5" y_distance="1.25" gazebo="true" two_cables="true" cable_distance="0.3"/>
 </robot>

File: schunk_lwa4p_description/urdf/powerline.xacro (robot description, xacro)
@@ -1,12 +1,12 @@
 <?xml version="1.0" encoding="utf-8"?>
 <robot xmlns:xacro="http://www.ros.org/wiki/xacro" name="powerline">
-    <xacro:macro name="powerline" params="base_x:=0 base_y:=0 base_z:=0 x_distance:=0.75 y_distance:=1 two_cables:=true gazebo:=true cable_distance=0.25">
+    <xacro:macro name="powerline" params="base_x:=0 base_y:=0 powerline_height:=0 x_distance:=0.75 y_distance:=1 two_cables:=true gazebo:=true cable_distance=0.25">
       <xacro:arg name="gazebo" default="true"/>
             <xacro:if value="$(arg gazebo)">
             <!-- Gazebo Tags -->
-                <xacro:include filename="$(find schunk_lwa4p_moveit)/urdf/powerline.gazebo.xacro"/>
+                <xacro:include filename="$(find schunk_lwa4p_description)/urdf/powerline.gazebo.xacro"/>
             </xacro:if>
         <joint name="base_powerline_link1" type="fixed">
-            <origin xyz="${x_distance} -${y_distance} 0.375" rpy="0 0 0"/>
+            <origin xyz="${x_distance} -${y_distance} ${powerline_height/2}" rpy="0 0 0"/>
             <parent link="base_link"/>
             <child link="powerline_link1"/>
@@ -17,5 +17,5 @@
 		        <origin xyz="0 0 0" rpy="0 0 0" />
 		        <geometry>
-			        <cylinder radius="0.05" length="0.75"/>
+			        <cylinder radius="0.05" length="${powerline_height}"/>
 		        </geometry>
 		        <material name="Gazebo/WoodFloor" />
@@ -24,5 +24,5 @@
 		        <origin xyz="0 0 0" rpy="0 0 0" />
 		        <geometry>
-		            <cylinder radius="0.1" length="0.75"/>
+		            <cylinder radius="0.01" length="${powerline_height}"/>
 		        </geometry>
 		    </collision>
@@ -34,5 +34,5 @@
 	    </link>
         <joint name="base_powerline_link2"  type="fixed">
-            <origin xyz="${x_distance} ${y_distance} 0.375" rpy="0 0 0"/>
+            <origin xyz="${x_distance} ${y_distance} ${powerline_height/2}" rpy="0 0 0"/>
             <parent link="base_link"/>
             <child link="powerline_link2"/>
@@ -42,5 +42,5 @@
 		   <origin xyz="0 0 0" rpy="0 0 0" />
 		   <geometry>
-			  <cylinder radius="0.05" length="0.75"/>
+			  <cylinder radius="0.05" length="${powerline_height}"/>
 		   </geometry>
 		   <material name="Gazebo/WoodFloor" />
@@ -49,5 +49,5 @@
 		   <origin xyz="0 0 0" rpy="0 0 0" />
 		   <geometry>
-			  <cylinder radius="0.05" length="0.75"/>
+			  <cylinder radius="0.05" length="${powerline_height}"/>
 		   </geometry>
 		</collision>
@@ -59,5 +59,5 @@
 	</link>
     <joint name="base_powerline_cable1" type="fixed">
-        <origin xyz="${x_distance} 0 0.75" rpy="0 0 0"/>
+        <origin xyz="${x_distance} 0 ${powerline_height}" rpy="0 0 0"/>
         <parent link="base_link"/>
         <child link="powerline_cable1"/>
@@ -85,5 +85,5 @@
     <xacro:if value="${two_cables}">
         <joint name="base_powerline_link3" type="fixed">
-            <origin xyz="${x_distance + cable_distance} -${y_distance} 0.375" rpy="0 0 0"/>
+            <origin xyz="${x_distance + cable_distance} -${y_distance} ${powerline_height/2}" rpy="0 0 0"/>
             <parent link="base_link"/>
             <child link="powerline_link3"/>
@@ -93,5 +93,5 @@
 		        <origin xyz="0 0 0" rpy="0 0 0" />
 		        <geometry>
-			        <cylinder radius="0.05" length="0.75"/>
+			        <cylinder radius="0.05" length="${powerline_height}"/>
 		        </geometry>
 		        <material name="Gazebo/WoodFloor" />
@@ -100,5 +100,5 @@
 		        <origin xyz="0 0 0" rpy="0 0 0" />
 		        <geometry>
-		            <cylinder radius="0.05" length="0.75"/>
+		            <cylinder radius="0.05" length="${powerline_height}"/>
 		        </geometry>
 		    </collision>
@@ -110,5 +110,5 @@
 	    </link>
         <joint name="base_powerline_link4" type="fixed">
-            <origin xyz="${x_distance + cable_distance} ${y_distance} 0.375" rpy="0 0 0"/>
+            <origin xyz="${x_distance + cable_distance} ${y_distance} ${powerline_height/2}" rpy="0 0 0"/>
             <parent link="base_link"/>
             <child link="powerline_link4"/>
@@ -118,5 +118,5 @@
                 <origin xyz="0 0 0" rpy="0 0 0" />
                 <geometry>
-                    <cylinder radius="0.05" length="0.75"/>
+                    <cylinder radius="0.05" length="${powerline_height}"/>
                 </geometry>
                 <material name="Gazebo/WoodFloor" />
@@ -125,5 +125,5 @@
                 <origin xyz="0 0 0" rpy="0 0 0" />
                 <geometry>
-                    <cylinder radius="0.05" length="0.75"/>
+                    <cylinder radius="0.05" length="${powerline_height}"/>
                 </geometry>
             </collision>
@@ -135,5 +135,5 @@
 	    </link>
         <joint name="base_powerline_cable2" type="fixed">
-            <origin xyz="${x_distance + cable_distance} 0 0.75" rpy="0 0 0"/>
+            <origin xyz="${x_distance + cable_distance} 0 ${powerline_height}" rpy="0 0 0"/>
             <parent link="base_link"/>
             <child link="powerline_cable2"/>

Commit message: Added parametrized powerline and executing of dummy cartesian trajectory

File: schunk_lwa4p_description/urdf/lwa4p/lwa4p_arm_separator_powerline.urdf.xacro (robot description, xacro)
@@ -14,25 +14,31 @@
   <xacro:include filename="$(find schunk_lwa4p_description)/urdf/powerline.xacro"/>
   <xacro:include filename="$(find schunk_lwa4p_description)/urdf/common.xacro"/>
-    <!-- foot for arm -->
-	<link name="base_link">
-		<visual>
-		   <origin xyz="0 0 0.25" rpy="0 0 0" />
-		   <geometry>
-			  <cylinder radius="0.1" length="0.5"/>
-		   </geometry>
-		   <material name="Gazebo/Black" />
-		</visual>
-		<collision>
-		   <origin xyz="0 0 0.25" rpy="0 0 0" />
-		   <geometry>
-			  <cylinder radius="0.1" length="0.5"/>
-		   </geometry>
-		</collision>
-		<inertial>
-		   <origin xyz="0 0 0.25" rpy="0 0 0"/>
-		   <mass value="10000.0"/>
-		   <inertia ixx="10000.0"  ixy="0"  ixz="0" iyy="10000.0" iyz="0" izz="10000.0" />
-		</inertial>
-	</link>
+  <link name="world">
+  </link>
+  <joint name="world_base_joint" type="fixed">
+	<parent link="world"/>
+	<child link="base_link"/>
+  </joint>
+  <!-- foot for arm -->
+  <link name="base_link">
+	<visual>
+		<origin xyz="0 0 0.25" rpy="0 0 0" />
+		<geometry>
+			<cylinder radius="0.1" length="0.5"/>
+		</geometry>
+		<material name="Gazebo/Black" />
+	</visual>
+	<collision>
+		<origin xyz="0 0 0.25" rpy="0 0 0" />
+		<geometry>
+			<cylinder radius="0.1" length="0.5"/>
+		</geometry>
+	</collision>
+	<inertial>
+		<origin xyz="0 0 0.25" rpy="0 0 0"/>
+		<mass value="10000.0"/>
+		<inertia ixx="10000.0"  ixy="0"  ixz="0" iyy="10000.0" iyz="0" izz="10000.0" />
+	</inertial>
+  </link>
   <!-- arm -->
   <xacro:lwa4p_arm arm_id="lwa4p" parent="base_link" has_podest="true" >
@@ -44,4 +50,4 @@
   <xacro:separator_distancer ns="lwa4p" rpy="0 0 0" xyz="0 0 0.05"/>
   <!-- powerline -->
-  <xacro:powerline base_x="0" base_y="0" powerline_height="1.0" x_distance="0.5" y_distance="1.25" gazebo="true" two_cables="true" cable_distance="0.3"/>
+  <xacro:powerline base_x="0" base_y="0" powerline_height="1.1" x_distance="0.25" y_distance="1.25" gazebo="true" two_cables="true" cable_distance="0.3"/>
 </robot>

Commit message: Added config files for follow_joint_trajectory/real robot+moveit integration

File: schunk_lwa4p_description/urdf/lwa4p/lwa4p_arm_separator_powerline.urdf.xacro (robot description, xacro)
@@ -46,5 +46,5 @@
   </xacro:lwa4p_arm>
   <!-- tool -->
-  <xacro:separator ns="lwa4p" rpy="0 0 0" connected_to="lwa4p_link6" safety_distance="0.03"/>
+  <xacro:separator ns="lwa4p" rpy="0 0 ${pi/2}" connected_to="lwa4p_link6" safety_distance="0.03"/>
   <!-- separator distancer -->
   <xacro:separator_distancer ns="lwa4p" rpy="0 0 0" xyz="0 0 0.05"/>

File: schunk_lwa4p_description/urdf/powerline.xacro (robot description, xacro)
@@ -8,5 +8,5 @@
             </xacro:if>
         <joint name="base_powerline_link1" type="fixed">
-            <origin xyz="${x_distance} -${y_distance} ${powerline_height/2}" rpy="0 0 0"/>
+            <origin xyz="-${x_distance} -${y_distance} ${powerline_height/2}" rpy="0 0 -1.507"/>
             <parent link="base_link"/>
             <child link="powerline_link1"/>
@@ -34,5 +34,5 @@
 	    </link>
         <joint name="base_powerline_link2"  type="fixed">
-            <origin xyz="${x_distance} ${y_distance} ${powerline_height/2}" rpy="0 0 0"/>
+            <origin xyz="-${x_distance} ${y_distance} ${powerline_height/2}" rpy="0 0 -1.507"/>
             <parent link="base_link"/>
             <child link="powerline_link2"/>
@@ -59,5 +59,5 @@
 	</link>
     <joint name="base_powerline_cable1" type="fixed">
-        <origin xyz="${x_distance} 0 ${powerline_height}" rpy="0 0 0"/>
+        <origin xyz="-${x_distance} 0 ${powerline_height}" rpy="0 0 0"/>
         <parent link="base_link"/>
         <child link="powerline_cable1"/>
@@ -85,5 +85,5 @@
     <xacro:if value="${two_cables}">
         <joint name="base_powerline_link3" type="fixed">
-            <origin xyz="${x_distance + cable_distance} -${y_distance} ${powerline_height/2}" rpy="0 0 0"/>
+            <origin xyz="-${x_distance + cable_distance} -${y_distance} ${powerline_height/2}" rpy="0 0 0"/>
             <parent link="base_link"/>
             <child link="powerline_link3"/>
@@ -110,5 +110,5 @@
 	    </link>
         <joint name="base_powerline_link4" type="fixed">
-            <origin xyz="${x_distance + cable_distance} ${y_distance} ${powerline_height/2}" rpy="0 0 0"/>
+            <origin xyz="-${x_distance + cable_distance} ${y_distance} ${powerline_height/2}" rpy="0 0 0"/>
             <parent link="base_link"/>
             <child link="powerline_link4"/>
@@ -135,5 +135,5 @@
 	    </link>
         <joint name="base_powerline_cable2" type="fixed">
-            <origin xyz="${x_distance + cable_distance} 0 ${powerline_height}" rpy="0 0 0"/>
+            <origin xyz="-${x_distance + cable_distance} 0 ${powerline_height}" rpy="0 0 0"/>
             <parent link="base_link"/>
             <child link="powerline_cable2"/>

Commit message: Added homing position to srdf, hz to trajectory fix

File: schunk_lwa4p_description/urdf/lwa4p/lwa4p_arm_separator_powerline.urdf.xacro (robot description, xacro)
@@ -50,4 +50,4 @@
   <xacro:separator_distancer ns="lwa4p" rpy="0 0 0" xyz="0 0 0.05"/>
   <!-- powerline -->
-  <xacro:powerline base_x="0" base_y="0" powerline_height="1.195" x_distance="0.19" y_distance="1.25" gazebo="true" two_cables="true" cable_distance="0.4"/>
+  <xacro:powerline base_x="0" base_y="0" powerline_height="1.195" x_distance="0.125" y_distance="1.25" gazebo="true" two_cables="true" cable_distance="0.4"/>
 </robot>

File: schunk_lwa4p_description/urdf/tools/separator.xacro (robot description, xacro)
@@ -171,5 +171,5 @@
             <parent link="separator_base"/>
             <child link="imu1"/>
-            <origin xyz="0.1 0.3 -0.01" rpy="0 0 0"/>
+            <origin xyz="-0.1 0.3 -0.01" rpy="0 0 0"/>
         </joint>
         <link name="imu2">
@@ -195,5 +195,5 @@
             <parent link="separator_base"/>
             <child link="imu2"/>
-            <origin xyz="0.1 0.0 -0.01" rpy="0 0 0"/>
+            <origin xyz="-0.1 0.0 -0.01" rpy="0 0 0"/>
         </joint>
         <link name="imu3">
@@ -219,5 +219,5 @@
             <parent link="separator_base"/>
             <child link="imu3"/>
-            <origin xyz="0.1 -0.3 -0.01" rpy="0 0 0"/>
+            <origin xyz="-0.1 -0.3 -0.01" rpy="0 0 0"/>
         </joint>
     </xacro:macro>

Commit message: Getting IK for goal pose

File: schunk_lwa4p_description/urdf/lwa4p/lwa4p_arm_separator_powerline.urdf.xacro (robot description, xacro)
@@ -23,18 +23,18 @@
   <link name="base_link">
 	<visual>
-		<origin xyz="0 0 0.25" rpy="0 0 0" />
+		<origin xyz="0 0 0.4" rpy="0 0 0" />
 		<geometry>
-			<cylinder radius="0.1" length="0.5"/>
+			<cylinder radius="0.1" length="0.8"/>
 		</geometry>
 		<material name="Gazebo/Black" />
 	</visual>
 	<collision>
-		<origin xyz="0 0 0.25" rpy="0 0 0" />
+		<origin xyz="0 0 0.4" rpy="0 0 0" />
 		<geometry>
-			<cylinder radius="0.1" length="0.5"/>
+			<cylinder radius="0.1" length="0.8"/>
 		</geometry>
 	</collision>
 	<inertial>
-		<origin xyz="0 0 0.25" rpy="0 0 0"/>
+		<origin xyz="0 0 0.4" rpy="0 0 0"/>
 		<mass value="10000.0"/>
 		<inertia ixx="10000.0"  ixy="0"  ixz="0" iyy="10000.0" iyz="0" izz="10000.0" />
@@ -43,5 +43,5 @@
   <!-- arm -->
   <xacro:lwa4p_arm arm_id="lwa4p" parent="base_link" has_podest="true" >
-    <origin xyz="0 0 0.50" rpy="0 0 0" />
+    <origin xyz="0 0 0.8" rpy="0 0 0" />
   </xacro:lwa4p_arm>
   <!-- tool -->
@@ -50,4 +50,4 @@
   <xacro:separator_distancer ns="lwa4p" rpy="0 0 0" xyz="0 0 0.05"/>
   <!-- powerline -->
-  <xacro:powerline base_x="0" base_y="0" powerline_height="1.195" x_distance="0.2" y_distance="1.25" gazebo="true" two_cables="true" cable_distance="0.4"/>
+  <xacro:powerline base_x="0" base_y="0" powerline_height="1.45" x_distance="0.05" y_distance="1.25" gazebo="true" two_cables="true" cable_distance="0.4"/>
 </robot>

Commit message: Added bare arm config for trying out trajectory execution:

File: schunk_lwa4p_description/urdf/lwa4p/lwa4p_arm_separator_powerline.urdf.xacro (robot description, xacro)
@@ -50,4 +50,4 @@
   <xacro:separator_distancer ns="lwa4p" rpy="0 0 0" xyz="0 0 0.05"/>
   <!-- powerline -->
-  <xacro:powerline base_x="0" base_y="0" powerline_height="1.40" x_distance="0.15" y_distance="1.25" gazebo="true" two_cables="true" cable_distance="0.4"/>
+  <xacro:powerline base_x="0" base_y="0" powerline_height="1.39" x_distance="0.15" y_distance="1.25" gazebo="true" two_cables="true" cable_distance="0.4"/>
 </robot>

File: schunk_lwa4p_description/urdf/tools/separator.xacro (robot description, xacro)
@@ -221,4 +221,100 @@
             <origin xyz="-0.1 -0.27 -0.01" rpy="0 0 0"/>
         </joint>
+        <link name="addition1">
+            <intertial>
+                <origin rpy="0 0 0" xyz="0 0 0"/>
+                <mass value="0.01"/>
+                <inertia ixx="0.01" ixy="0.0" ixz="0.0" iyz="0.0" izz="0.01"/>
+            </intertial>
+            <visual>
+                <origin rpy="0 0 0" xyz="0 0 0"/>
+                <geometry>
+                    <box size="0.01 0.035 0.01"/>
+                </geometry>
+            </visual>
+            <collision>
+                <origin rpy="0 0 0" xyz="0 0 0"/>
+                <geometry>
+                    <box size="0.01 0.035 0.01"/>
+                </geometry>
+            </collision>
+        </link>
+        <joint name="separator_addition1" type="fixed">
+            <parent link="separator_base"/>
+            <child link="addition1"/>
+            <origin xyz="-0.05 -0.35 -0.01" rpy="0 0 0"/>
+        </joint>
+        <link name="addition2">
+            <intertial>
+                <origin rpy="0 0 0" xyz="0 0 0"/>
+                <mass value="0.01"/>
+                <inertia ixx="0.01" ixy="0.0" ixz="0.0" iyz="0.0" izz="0.01"/>
+            </intertial>
+            <visual>
+                <origin rpy="0 0 0" xyz="0 0 0"/>
+                <geometry>
+                    <box size="0.01 0.035 0.01"/>
+                </geometry>
+            </visual>
+            <collision>
+                <origin rpy="0 0 0" xyz="0 0 0"/>
+                <geometry>
+                    <box size="0.01 0.035 0.01"/>
+                </geometry>
+            </collision>
+        </link>
+        <joint name="separator_addition2" type="fixed">
+            <parent link="separator_base"/>
+            <child link="addition2"/>
+            <origin xyz="0.05 -0.35 -0.01" rpy="0 0 0"/>
+        </joint>
+        <link name="addition3">
+            <intertial>
+                <origin rpy="0 0 0" xyz="0 0 0"/>
+                <mass value="0.01"/>
+                <inertia ixx="0.01" ixy="0.0" ixz="0.0" iyz="0.0" izz="0.01"/>
+            </intertial>
+            <visual>
+                <origin rpy="0 0 0" xyz="0 0 0"/>
+                <geometry>
+                    <box size="0.01 0.035 0.01"/>
+                </geometry>
+            </visual>
+            <collision>
+                <origin rpy="0 0 0" xyz="0 0 0"/>
+                <geometry>
+                    <box size="0.01 0.035 0.01"/>
+                </geometry>
+            </collision>
+        </link>
+        <joint name="separator_addition3" type="fixed">
+            <parent link="separator_base"/>
+            <child link="addition3"/>
+            <origin xyz="0.05 0.35 -0.01" rpy="0 0 0"/>
+        </joint>
+        <link name="addition4">
+            <intertial>
+                <origin rpy="0 0 0" xyz="0 0 0"/>
+                <mass value="0.01"/>
+                <inertia ixx="0.01" ixy="0.0" ixz="0.0" iyz="0.0" izz="0.01"/>
+            </intertial>
+            <visual>
+                <origin rpy="0 0 0" xyz="0 0 0"/>
+                <geometry>
+                    <box size="0.01 0.035 0.01"/>
+                </geometry>
+            </visual>
+            <collision>
+                <origin rpy="0 0 0" xyz="0 0 0"/>
+                <geometry>
+                    <box size="0.01 0.035 0.01"/>
+                </geometry>
+            </collision>
+        </link>
+        <joint name="separator_addition4" type="fixed">
+            <parent link="separator_base"/>
+            <child link="addition4"/>
+            <origin xyz="-0.05 0.35 0.0" rpy="0 0 0"/>
+        </joint>
     </xacro:macro>
 </robot>
