Commit message: Added updated bare arm which runs

File: schunk_lwa4p_description/urdf/lwa4p/lwa4p_arm.urdf.xacro (robot description, xacro)
@@ -8,18 +8,18 @@
 	<link name="base_link">
 		<visual>
-		   <origin xyz="0 0 0.25" rpy="0 0 0" />
+		   <origin xyz="0 0 0.4" rpy="0 0 0" />
 		   <geometry>
-			  <cylinder radius="0.1" length="0.5"/>
+			  <cylinder radius="0.1" length="0.8"/>
 		   </geometry>
 		   <material name="Gazebo/DarkGrey" />
 		</visual>
 		<collision>
-		   <origin xyz="0 0 0.25" rpy="0 0 0" />
+		   <origin xyz="0 0 0.4" rpy="0 0 0" />
 		   <geometry>
-			  <cylinder radius="0.1" length="0.5"/>
+			  <cylinder radius="0.1" length="0.8"/>
 		   </geometry>
 		</collision>
 		<inertial>
-		   <origin xyz="0 0 0.25" rpy="0 0 0"/>
+		   <origin xyz="0 0 0.4" rpy="0 0 0"/>
 		   <mass value="10000.0"/>
 		   <inertia ixx="10000.0"  ixy="0"  ixz="0" iyy="10000.0" iyz="0" izz="10000.0" />
@@ -28,5 +28,5 @@
   <!-- arm -->
   <xacro:lwa4p_arm arm_id="lwa4p" parent="base_link" has_podest="true" >
-    <origin xyz="0 0 0.50" rpy="0 0 0" />
+    <origin xyz="0 0 0.8" rpy="0 0 0" />
   </xacro:lwa4p_arm>
 </robot>

Commit message: A bunch of stuff to get the lab to work

File: schunk_lwa4p_description/urdf/lwa4p/lwa4p_arm.urdf.xacro (robot description, xacro)
@@ -8,18 +8,18 @@
 	<link name="base_link">
 		<visual>
-		   <origin xyz="0 0 0.4" rpy="0 0 0" />
+		   <origin xyz="0 0 0.5" rpy="0 0 0" />
 		   <geometry>
-			  <cylinder radius="0.1" length="0.8"/>
+			  <cylinder radius="0.1" length="1.0"/>
 		   </geometry>
 		   <material name="Gazebo/DarkGrey" />
 		</visual>
 		<collision>
-		   <origin xyz="0 0 0.4" rpy="0 0 0" />
+		   <origin xyz="0 0 0.5" rpy="0 0 0" />
 		   <geometry>
-			  <cylinder radius="0.1" length="0.8"/>
+			  <cylinder radius="0.1" length="1.0"/>
 		   </geometry>
 		</collision>
 		<inertial>
-		   <origin xyz="0 0 0.4" rpy="0 0 0"/>
+		   <origin xyz="0 0 0.5" rpy="0 0 0"/>
 		   <mass value="10000.0"/>
 		   <inertia ixx="10000.0"  ixy="0"  ixz="0" iyy="10000.0" iyz="0" izz="10000.0" />
@@ -28,5 +28,5 @@
   <!-- arm -->
   <xacro:lwa4p_arm arm_id="lwa4p" parent="base_link" has_podest="true" >
-    <origin xyz="0 0 0.8" rpy="0 0 0" />
+    <origin xyz="0 0 1.0" rpy="0 0 0" />
   </xacro:lwa4p_arm>
 </robot>

File: schunk_lwa4p_description/urdf/lwa4p/lwa4p_arm.xacro (robot description, xacro)
@@ -207,5 +207,5 @@
     <!-- joint between arm_4_link and arm_5_link -->
     <joint name="${arm_id}_joint5" type="revolute">
-      <origin xyz="0 0.005263 0.305" rpy="1.5708 0 3.14159" />
+      <origin xyz="0 0.0 0.305" rpy="1.5708 0 3.14159" />
       <parent link="${arm_id}_link4"/>
       <child link="${arm_id}_link5"/>

File: schunk_lwa4p_description/urdf/lwa4p/lwa4p_arm_wsg50.urdf.xacro (robot description, xacro)
@@ -17,18 +17,18 @@
     <link name="base_link">
         <visual>
-            <origin xyz="0 0 0.4" rpy="0 0 0" />
+            <origin xyz="0 0 0.5" rpy="0 0 0" />
             <geometry>
-                <cylinder radius="0.1" length="0.8"/>
+                <cylinder radius="0.1" length="1.0"/>
             </geometry>
             <material name="Gazebo/Black" />
         </visual>
         <collision>
-            <origin xyz="0 0 0.4" rpy="0 0 0" />
+            <origin xyz="0 0 0.5" rpy="0 0 0" />
             <geometry>
-                <cylinder radius="0.1" length="0.8"/>
+                <cylinder radius="0.1" length="1.0"/>
             </geometry>
         </collision>
         <inertial>
-            <origin xyz="0 0 0.4" rpy="0 0 0"/>
+            <origin xyz="0 0 0.5" rpy="0 0 0"/>
             <mass value="10000.0"/>
             <inertia ixx="10000.0"  ixy="0"  ixz="0" iyy="10000.0" iyz="0" izz="10000.0" />
@@ -37,8 +37,8 @@
     <!-- arm -->
     <xacro:lwa4p_arm arm_id="lwa4p" parent="base_link" has_podest="true" >
-        <origin xyz="0 0 0.8" rpy="0 0 0" />
+        <origin xyz="0 0 1.05" rpy="0 0 0" />
     </xacro:lwa4p_arm>
     <!-- wsg 50 gripper -->
-    <xacro:wsg_50_xacro name="wsg50" parent="lwa4p_link6" finger_length="0.1" finger_tip="0" off_dist="0.085" rotation="${pi/2}" >
+    <xacro:wsg_50_xacro name="wsg50" parent="lwa4p_link6" finger_length="0.1" finger_tip="0.08" off_dist="0.085" rotation="${pi/2}" >
         <origin xyz="0 0 0" rpy="0 0 0" />
     </xacro:wsg_50_xacro>

File: schunk_lwa4p_description/urdf/tools/wsg50.urdf.xacro (robot description, xacro)
@@ -47,5 +47,5 @@
   </gazebo>
   <joint name="${name}_center_joint" type="fixed">
-     <origin xyz="0 0 ${finger_length}" rpy="0 0 0" />      <!--origin xyz="-0.0067 0 0.049" rpy="0 0 0" /-->
+     <origin xyz="0 0 0.2" rpy="0 0 0" />      <!--origin xyz="-0.0067 0 0.049" rpy="0 0 0" /-->
      <parent link="${name}_base_link"/>
      <child link="${name}_center" />
@@ -63,9 +63,13 @@
      <limit effort="100" velocity="100"/>
   </joint>
-  <transmission name="${name}_base_trans_left" type="pr2_mechanism_model/SimpleTransmission">
-     <actuator name="${name}_base_motor_left" />
-     <joint name="${name}_base_joint_gripper_left" />
-     <mechanicalReduction>1</mechanicalReduction>
-     <motorTorqueConstant>1</motorTorqueConstant>
+  <transmission name="${name}_finger_left_joint_trans">
+    <type>transmission_interface/SimpleTransmission</type>
+    <joint name="${name}_finger_left_joint">
+      <hardwareInterface>hardware_interface/PositionJointInterface</hardwareInterface>
+      <!--hardwareInterface>hardware_interface/VelocityJointInterface</hardwareInterface!-->
+    </joint>
+    <actuator name="${name}_finger_left_joint_motor">
+      <mechanicalReduction>1</mechanicalReduction>
+    </actuator>
   </transmission>
   <link name="${name}_gripper_left">
@@ -148,9 +152,13 @@
      <limit effort="100" velocity="100"/>
   </joint>
-  <transmission name="${name}_base_trans_right" type="pr2_mechanism_model/SimpleTransmission">
-     <actuator name="${name}_base_motor_right" />
-     <joint name="${name}_base_joint_gripper_right" />
-     <mechanicalReduction>1</mechanicalReduction>
-     <motorTorqueConstant>1</motorTorqueConstant>
+ <transmission name="${name}_finger_right_joint_trans">
+    <type>transmission_interface/SimpleTransmission</type>
+    <joint name="${name}_finger_right_joint">
+      <hardwareInterface>hardware_interface/PositionJointInterface</hardwareInterface>
+      <!--hardwareInterface>hardware_interface/VelocityJointInterface</hardwareInterface!-->
+    </joint>
+    <actuator name="${name}_finger_right_joint_motor">
+      <mechanicalReduction>1</mechanicalReduction>
+    </actuator>
   </transmission>
     <link name="${name}_gripper_right">
