Commit message: Added some changes for Christmas 22!

File: schunk_lwa4p_description/urdf/lwa4p/lwa4p_arm_wsg50.urdf.xacro (robot description, xacro)
@@ -17,18 +17,18 @@
     <link name="base_link">
         <visual>
-            <origin xyz="0 0 0.4" rpy="0 0 0" />
+            <origin xyz="0 0 0.125" rpy="0 0 0" />
             <geometry>
-                <cylinder radius="0.1" length="0.8"/>
+                <cylinder radius="0.1" length="0.25"/>
             </geometry>
             <material name="Gazebo/Black" />
         </visual>
         <collision>
-            <origin xyz="0 0 0.4" rpy="0 0 0" />
+            <origin xyz="0 0 0.125" rpy="0 0 0" />
             <geometry>
-                <cylinder radius="0.1" length="0.8"/>
+                <cylinder radius="0.1" length="0.25"/>
             </geometry>
         </collision>
         <inertial>
-            <origin xyz="0 0 0.4" rpy="0 0 0"/>
+            <origin xyz="0 0 0.125" rpy="0 0 0"/>
             <mass value="10000.0"/>
             <inertia ixx="10000.0"  ixy="0"  ixz="0" iyy="10000.0" iyz="0" izz="10000.0" />
@@ -37,5 +37,5 @@
     <!-- arm -->
     <xacro:lwa4p_arm arm_id="lwa4p" parent="base_link" has_podest="true" >
-        <origin xyz="0 0 0.8" rpy="0 0 0" />
+        <origin xyz="0 0 0.25" rpy="0 0 0" />
     </xacro:lwa4p_arm>
     <!-- wsg 50 gripper -->

Commit message: [Christmas ready] Bogu hvala!

File: schunk_lwa4p_description/urdf/lwa4p/lwa4p_arm_wsg50.urdf.xacro (robot description, xacro)
@@ -17,18 +17,18 @@
     <link name="base_link">
         <visual>
-            <origin xyz="0 0 0.125" rpy="0 0 0" />
+            <origin xyz="0 0 0.0" rpy="0 0 0" />
             <geometry>
-                <cylinder radius="0.1" length="0.25"/>
+                <cylinder radius="0.0" length="0.0"/>
             </geometry>
             <material name="Gazebo/Black" />
         </visual>
         <collision>
-            <origin xyz="0 0 0.125" rpy="0 0 0" />
+            <origin xyz="0 0 0.0" rpy="0 0 0" />
             <geometry>
-                <cylinder radius="0.1" length="0.25"/>
+                <cylinder radius="0.0" length="0.0"/>
             </geometry>
         </collision>
         <inertial>
-            <origin xyz="0 0 0.125" rpy="0 0 0"/>
+            <origin xyz="0 0 0.0" rpy="0 0 0"/>
             <mass value="10000.0"/>
             <inertia ixx="10000.0"  ixy="0"  ixz="0" iyy="10000.0" iyz="0" izz="10000.0" />
@@ -37,5 +37,5 @@
     <!-- arm -->
     <xacro:lwa4p_arm arm_id="lwa4p" parent="base_link" has_podest="true" >
-        <origin xyz="0 0 0.25" rpy="0 0 0" />
+        <origin xyz="0 0 0.1" rpy="0 0 0" />
     </xacro:lwa4p_arm>
     <!-- wsg 50 gripper -->

Commit message: Added some changes for real robot execution

File: schunk_lwa4p_description/urdf/lwa4p/lwa4p_arm_wsg50.urdf.xacro (robot description, xacro)
@@ -17,18 +17,18 @@
     <link name="base_link">
         <visual>
-            <origin xyz="0 0 0.5" rpy="0 0 0" />
+            <origin xyz="0 0 0.3" rpy="0 0 0" />
             <geometry>
-                <cylinder radius="0.1" length="1.0"/>
+                <cylinder radius="0.1" length="0.6"/>
             </geometry>
             <material name="Gazebo/Black" />
         </visual>
         <collision>
-            <origin xyz="0 0 0.5" rpy="0 0 0" />
+            <origin xyz="0 0 0.3" rpy="0 0 0" />
             <geometry>
-                <cylinder radius="0.1" length="1.0"/>
+                <cylinder radius="0.1" length="0.6"/>
             </geometry>
         </collision>
         <inertial>
-            <origin xyz="0 0 0.5" rpy="0 0 0"/>
+            <origin xyz="0 0 0.3" rpy="0 0 0"/>
             <mass value="10000.0"/>
             <inertia ixx="10000.0"  ixy="0"  ixz="0" iyy="10000.0" iyz="0" izz="10000.0" />
@@ -37,5 +37,5 @@
     <!-- arm -->
     <xacro:lwa4p_arm arm_id="lwa4p" parent="base_link" has_podest="true" >
-        <origin xyz="0 0 1.05" rpy="0 0 0" />
+        <origin xyz="0 0 0.6" rpy="0 0 0" />
     </xacro:lwa4p_arm>
     <!-- wsg 50 gripper -->
