Commit message: Added IMUs to separator model to enable collision check and mitigate possible collisions when using real robot.

File: schunk_lwa4p_description/urdf/tools/separator.gazebo.xacro (robot description, xacro)
@@ -15,4 +15,13 @@
     <gazebo reference="separator_left_front_holder">
         <material value="Gazebo/Green" />
+    </gazebo>
+    <gazebo reference="imu1">
+        <material value="Gazebo/Blue"/>
+    </gazebo>
+    <gazebo reference="imu2">
+        <material value="Gazebo/Blue"/>
+    </gazebo>
+    <gazebo reference="imu3">
+        <material value="Gazebo/Blue"/>
     </gazebo>
     <transmission name="separator_right_front_trans">

File: schunk_lwa4p_description/urdf/tools/separator.xacro (robot description, xacro)
@@ -148,4 +148,77 @@
             <axis xyz="0 1 0"/>
         </joint>
+        <!-- Add IMUs to mitiagate possible collision !-->
+        <link name="imu1">
+            <intertial>
+                <origin rpy="0 0 0" xyz="0 0 0"/>
+                <mass value="0.01"/>
+                <inertia ixx="0.01" ixy="0.0" ixz="0.0" iyz="0.0" izz="0.01"/>
+            </intertial>
+            <visual>
+                <origin rpy="0 0 0" xyz="0 0 0"/>
+                <geometry>
+                    <box size="0.05 0.05 0.02"/>
+                </geometry>
+            </visual>
+            <collision>
+                <origin rpy="0 0 0" xyz="0 0 0"/>
+                <geometry>
+                    <box size="0.05 0.05 0.02"/>
+                </geometry>
+            </collision>
+        </link>
+        <joint name="separator_imu1" type="fixed">
+            <parent link="separator_base"/>
+            <child link="imu1"/>
+            <origin xyz="0.1 0.3 -0.01" rpy="0 0 0"/>
+        </joint>
+        <link name="imu2">
+            <intertial>
+                <origin rpy="0 0 0" xyz="0 0 0"/>
+                <mass value="0.01"/>
+                <inertia ixx="0.01" ixy="0.0" ixz="0.0" iyz="0.0" izz="0.01"/>
+            </intertial>
+            <visual>
+                <origin rpy="0 0 0" xyz="0 0 0"/>
+                <geometry>
+                    <box size="0.05 0.05 0.02"/>
+                </geometry>
+            </visual>
+            <collision>
+                <origin rpy="0 0 0" xyz="0 0 0"/>
+                <geometry>
+                    <box size="0.05 0.05 0.02"/>
+                </geometry>
+            </collision>
+        </link>
+        <joint name="separator_imu2" type="fixed">
+            <parent link="separator_base"/>
+            <child link="imu2"/>
+            <origin xyz="0.1 0.0 -0.01" rpy="0 0 0"/>
+        </joint>
+        <link name="imu3">
+            <intertial>
+                <origin rpy="0 0 0" xyz="0 0 0"/>
+                <mass value="0.01"/>
+                <inertia ixx="0.01" ixy="0.0" ixz="0.0" iyz="0.0" izz="0.01"/>
+            </intertial>
+            <visual>
+                <origin rpy="0 0 0" xyz="0 0 0"/>
+                <geometry>
+                    <box size="0.05 0.05 0.02"/>
+                </geometry>
+            </visual>
+            <collision>
+                <origin rpy="0 0 0" xyz="0 0 0"/>
+                <geometry>
+                    <box size="0.05 0.05 0.02"/>
+                </geometry>
+            </collision>
+        </link>
+        <joint name="separator_imu3" type="fixed">
+            <parent link="separator_base"/>
+            <child link="imu3"/>
+            <origin xyz="0.1 -0.3 -0.01" rpy="0 0 0"/>
+        </joint>
     </xacro:macro>
 </robot>
