Commit message: Added IMU measurements bagging script and StatusMonitor to servoing

File: schunk_lwa4p_description/urdf/tools/separator.xacro (robot description, xacro)
@@ -171,5 +171,5 @@
             <parent link="separator_base"/>
             <child link="imu1"/>
-            <origin xyz="-0.1 0.3 -0.01" rpy="0 0 0"/>
+            <origin xyz="-0.1 0.27 -0.01" rpy="0 0 0"/>
         </joint>
         <link name="imu2">
@@ -219,5 +219,5 @@
             <parent link="separator_base"/>
             <child link="imu3"/>
-            <origin xyz="-0.1 -0.3 -0.01" rpy="0 0 0"/>
+            <origin xyz="-0.1 -0.27 -0.01" rpy="0 0 0"/>
         </joint>
     </xacro:macro>
